File: DropDN - redesign plate making.kicad_pcb (KiCad board)
At the start: 2 copper layers, 878.7 x 316.7 mm, 70 parts

Commit message: idk, some changes maybe
Parts:
- moved RESET1 56.8 mm to (-600.1, 129.8)
Other:
- board size 878.7 x 316.7 mm -> 935.2 x 316.7 mm

Commit message: bunch of updates
1) Made 3 small modifications to the case design based on the proto:
a) more clearance for switches on top layer
b) actual clearance for usb port on PM
c) closed the compression layer for aesthetics

2) made alterations to the PCB silk

3) fixed an issue with the reset switch pads that prevented a physically soldered reset switch from working
Parts:
- removed the RESET1 at (-600.1, 129.8)
Other:
- board size 935.2 x 316.7 mm -> 793.6 x 316.7 mm
