File: DropDN - redesign plate making.kicad_pcb (KiCad board)
At the start: 2 copper layers, 793.6 x 316.7 mm, 69 parts

Commit message: updated case files
Parts:
- added RESET1: reset, random-keyboard-parts:SKQG-1155865, B.Cu at (-58.9, 336.9)
Other:
- board size 793.6 x 316.7 mm -> 793.6 x 427.4 mm

Commit message: huge overhaul
Parts:
- moved RESET1 426.8 mm to (156.9, 137.5)
Other:
- board size 793.6 x 427.4 mm -> 803.4 x 427.4 mm
