File: DropDN - redesign.kicad_pcb (KiCad board)
At the start: 2 copper layers, 171.5 x 76.2 mm, 70 parts

Commit message: bunch of updates
1) Made 3 small modifications to the case design based on the proto:
a) more clearance for switches on top layer
b) actual clearance for usb port on PM
c) closed the compression layer for aesthetics

2) made alterations to the PCB silk

3) fixed an issue with the reset switch pads that prevented a physically soldered reset switch from working
Parts:
- removed the G*** at (158.4, 49.4)
- moved G*** 32.3 mm to (75.2, 82.0)
Other:
- board text added: "A"
- board text added: "A Modified Colemak Layout by: DrHigsby"
- board text added: "B"
- board text added: "C"
- board text added: "D"
- board text added: "E"
- board text added: "F"
- board text added: "G"
- board text added: "H"
- board text added: "I"
- board text added: "J"
- board text added: "K"
- board text added: "KC_COMM"
- board text added: "KC_DOT"
- board text added: "KC_LCTL"
- board text added: "KC_RALT"
- board text added: "KC_SLSH"
- board text added: "KC_SPC"
- board text added: "L"
- board text added: "M"
- board text added: "MO(1)"
- board text added: "N"
- board text added: "O"
- board text added: "P"
- board text added: "Q"
- board text added: "R"
- board text added: "S"
- board text added: "T"
- board text added: "U"
- board text added: "V"
- board text added: "W"
- board text added: "X"
- board text added: "Y"
- board text added: "Z"
